Commit message: Changed Mass and length properties. Added Inertial macro. Changed effort to 1.96Nm (20kg per cm). Added Odom, encoder etc values to plugin. Changed Max angular and linear speed. Added PID values for position controller

File: description/robot_core.xacro (robot description, xacro)
@@ -6,9 +6,9 @@
 <robot xmlns:xacro="http://www.ros.org/wiki/xacro" name="tracked_robot_2">
 	<xacro:include filename="inertial_macros.xacro" />
-	<xacro:property name="mass" value="15"> </xacro:property>
-    <xacro:property name="base_mass" value="15" />
-    <xacro:property name="track_mass" value="10" />
-    <xacro:property name="flipper_mass" value="2.5" />
-    <xacro:property name="flipper_length" value="0.139577" />
+	<xacro:property name="mass" value="1.5"> </xacro:property>
+    <xacro:property name="base_mass" value="1.50" />
+    <xacro:property name="track_mass" value="0." />
+    <xacro:property name="flipper_mass" value="0.375" />
+    <xacro:property name="flipper_length" value="0.025" />
 	<!-- BASE LINK -->
 	<link name="base_link">
@@ -21,8 +21,12 @@
 	<!-- CHASSIS LINK -->
 	<link name="chassis_link">
-		<!-- <xacro:inertial_box mass="${mass}" x="0.25932" y="0.153" z="0.05932">
+<!--
+		<xacro:inertial_box mass="${mass}" x="0.25932" y="0.153" z="0.05932">
 			<origin xyz="1.5315E-06 -1.1582E-06 0.024757" rpy="0 0 0" />
 		</xacro:inertial_box> -->
-        <inertial>
+		<xacro:inertial_box mass="${mass}" x="0.25932" y="0.153" z="0.05932">
+			<origin xyz="0 0 0.024757" rpy="0 0 0" />
+		</xacro:inertial_box>
+        <!-- <inertial>
 			<origin xyz="0 0 0.024757" rpy="0 0 0" />
 			<mass
@@ -35,5 +39,5 @@
 			iyz="0"
 			izz="5" />
-        </inertial>
+        </inertial> -->
 		<visual>
 			<origin xyz="0 0 0" rpy="0 0 0" />
@@ -57,8 +61,8 @@
 	</gazebo>
 	<link name="imu_link">
-		<!-- <xacro:inertial_box mass="${mass}" x="0.25932" y="0.153" z="0.05932">
+		<xacro:inertial_box mass="${mass}" x="0.25932" y="0.153" z="0.05932">
 			<origin xyz="1.5315E-06 -1.1582E-06 0.024757" rpy="0 0 0" />
-		</xacro:inertial_box> -->
-        <inertial>
+		</xacro:inertial_box>
+        <!-- <inertial>
 			<origin xyz="0 0 0.024757" rpy="0 0 0" />
 			<mass
@@ -71,5 +75,5 @@
 			iyz="0"
 			izz="5" />
-        </inertial>
+        </inertial> -->
 		<visual>
 			<origin xyz="0 0 0" rpy="0 0 0" />
@@ -117,9 +121,8 @@
 	<!-- LEFT FLIPPER LINK -->
 	<link name="left_flipper_link">
-<!--
 		<xacro:inertial_box mass="${flipper_mass}" x="0.139577" y="0.045" z="0.06958">
 			<origin xyz="0.033943 0.00023886 0.011429" rpy="0 0 0" />
-		</xacro:inertial_box> -->
-        <inertial>
+		</xacro:inertial_box>
+        <!-- <inertial>
             <origin xyz="0.034059 0.0 -0.0" rpy="0 0 0" />
             <mass
@@ -132,5 +135,5 @@
 		iyz="0"
 		izz="5" />
-        </inertial>
+        </inertial> -->
 		<visual>
 			<origin xyz="0 0 0" rpy="0 0 0" />
@@ -151,5 +154,5 @@
 		<child link="left_flipper_link" />
 		<axis xyz="0 0 1" />
-		<limit lower="-3" upper="3" effort="0.5" velocity="1.0" />
+		<limit lower="-3" upper="3" effort="1.96" velocity="1.0" />
 	</joint>
 	<gazebo reference="left_flipper_link">
@@ -163,8 +166,8 @@
 	<!-- LEFT FLIPPER LINK -->
 	<link name="right_flipper_link">
-		<!-- <xacro:inertial_box mass="${flipper_mass}" x="0.139577" y="0.045" z="0.06958">
+		<xacro:inertial_box mass="${flipper_mass}" x="0.139577" y="0.045" z="0.06958">
 			<origin xyz="0.034069 7.9651E-05 -0.00043099" rpy="0 0 0" />
-		</xacro:inertial_box> -->
-        <inertial>
+		</xacro:inertial_box>
+        <!-- <inertial>
             <origin xyz="0.034069 0 -0.0" rpy="0 0 0" />
             <mass
@@ -177,5 +180,5 @@
 		iyz="0"
 		izz="5" />
-        </inertial>
+        </inertial> -->
 		<visual>
 			<origin xyz="0 0 0" rpy="0 0 0" />
@@ -196,5 +199,5 @@
 		<child link="right_flipper_link" />
 		<axis xyz="0 0 1" />
-		<limit lower="-3" upper="3" effort="0.5" velocity="1.0" />
+		<limit lower="-3" upper="3" effort="1.96" velocity="1.0" />
 	</joint>
 	<gazebo reference="right_flipper_link">
@@ -208,8 +211,8 @@
 	<!-- LEFT FLIPPER LINK -->
 	<link name="rear_left_flipper_link">
-		<!-- <xacro:inertial_box mass="${flipper_mass}" x="0.139577" y="0.045" z="0.06958">
+		<xacro:inertial_box mass="${flipper_mass}" x="0.139577" y="0.045" z="0.06958">
 			<origin xyz="-0.033863 -3.5938E-05 -0.00043099" rpy="0 0 0" />
-		</xacro:inertial_box> -->
-        <inertial>
+		</xacro:inertial_box>
+        <!-- <inertial>
             <origin xyz="-0.033863 0 0" rpy="0 0 0" />
             <mass
@@ -222,5 +225,5 @@
 		iyz="0"
 		izz="5" />
-        </inertial>
+        </inertial> -->
 		<visual>
 			<origin xyz="0 0 0" rpy="0 0 0" />
@@ -241,5 +244,5 @@
 		<child link="rear_left_flipper_link" />
 		<axis xyz="0 0 1" />
-		<limit lower="-3" upper="3" effort="0.5" velocity="1.0" />
+		<limit lower="-3" upper="3" effort="1.96" velocity="1.0" />
 	</joint>
 	<gazebo reference="rear_left_flipper_link">
@@ -253,9 +256,8 @@
 		<!-- LEFT FLIPPER LINK -->
 		<link name="rear_right_flipper_link">
-			<!-- <xacro:inertial_box mass="${flipper_mass}" x="0.139577" y="0.045" z="0.06958">
+			<xacro:inertial_box mass="${flipper_mass}" x="0.139577" y="0.045" z="0.06958">
 			<origin xyz="0.033863 7.9651E-05 -0.00043099" rpy="0 0 0" />
 			</xacro:inertial_box>
-	 -->
-	 <inertial>
+	 <!-- <inertial>
 		<origin xyz="-0.034063 -0.0 -0.0" rpy="0 0 0" />
 		<mass
@@ -268,5 +270,5 @@
 		iyz="0"
 		izz="5" />
-	</inertial>
+	</inertial> -->
 			<visual>
 				<origin xyz="0 0 0" rpy="0 0 0" />
@@ -287,5 +289,5 @@
 			<child link="rear_right_flipper_link" />
 			<axis xyz="0 0 1" />
-			<limit lower="-3" upper="3" effort="0.5" velocity="1.0" />
+			<limit lower="-3" upper="3" effort="1.96" velocity="1.0" />
 		</joint>
 		<gazebo reference="rear_right_flipper_link">
@@ -321,6 +323,10 @@
 			<commandROSTopic>/cmd_vel</commandROSTopic>
 			<commandIGNTopic>~/tracked_robot_2/cmd_vel_twist</commandIGNTopic>
-			<robotBaseFrame>base_link</robotBaseFrame>
+			<odometryTopic>odom</odometryTopic> <!-- ROS topic for the odometry data - remap if you're using another odom source -->
+			<robotBaseFrame>chassis_link</robotBaseFrame>
 			<tracks_separation>0.571</tracks_separation>
+			<publishOdomTF>true</publishOdomTF>
+			<odometrySource>encoder</odometrySource> <!-- [encoder,world] - choose world for ground truth -->
+			<trackSpeedTopic>~/tracked_robot_2/tracks_speed</trackSpeedTopic>
 		</plugin>
 	</gazebo>
@@ -337,6 +343,6 @@
 			<track_mu>2</track_mu>
 			<track_mu2>0.5</track_mu2>
-			<max_angular_speed>0.1</max_angular_speed>
-			<max_linear_speed>0.1</max_linear_speed>
+			<max_angular_speed>1.0</max_angular_speed>
+			<max_linear_speed>1.0</max_linear_speed>
 		</plugin>
 	</gazebo>
@@ -356,18 +362,81 @@
 		</plugin>
 	</gazebo>
-	    <!-- <ros2_control name="GazeboSystem" type="system">
+	<!-- <gazebo>
+		<plugin name="rotational_joint_control" filename="libgazebo_ros2_control.so">
+			<joint_name>left_flipper_joint</joint_name>
+		</plugin>
+	</gazebo> -->
+	<ros2_control name="GazeboSystem" type="system">
         <hardware>
             <plugin>gazebo_ros2_control/GazeboSystem</plugin>
         </hardware>
-    <joint name="left_flipper_joint">
-        <command_interface name="position">
-        </command_interface>
-        <state_interface name="position"/>
-        <state_interface name="velocity"/>
-      </joint>
+		<joint name="left_flipper_joint">
+			<param name="pos_kp">10.0001</param>
+			<param name="pos_ki">1.01</param>
+			<param name="pos_kd">1.01</param>
+			<param name="pos_max_integral_error">0.1</param>
+			<command_interface name="position_pid">
+				<param name="min">-3.0</param>
+				<param name="max">3.0</param>
+				</command_interface>
+			<state_interface name="position"/>
+			<state_interface name="effort"/>
+			<state_interface name="velocity"/>
+      	</joint>
+		  <joint name="right_flipper_joint">
+			<param name="pos_kp">10.0001</param>
+			<param name="pos_ki">1.01</param>
+			<param name="pos_kd">1.01</param>
+			<param name="pos_max_integral_error">0.1</param>
+			<command_interface name="position_pid">
+				<param name="min">-3.0</param>
+				<param name="max">3.0</param>
+				</command_interface>
+			<state_interface name="position"/>
+			<state_interface name="effort"/>
+			<state_interface name="velocity"/>
+      	</joint>
+		  <joint name="rear_left_flipper_joint">
+			<param name="pos_kp">10.0001</param>
+			<param name="pos_ki">1.01</param>
+			<param name="pos_kd">1.01</param>
+			<param name="pos_max_integral_error">0.1</param>
+			<command_interface name="position_pid">
+				<param name="min">-3.0</param>
+				<param name="max">3.0</param>
+				</command_interface>
+			<state_interface name="position"/>
+			<state_interface name="effort"/>
+			<state_interface name="velocity"/>
+      	</joint>
+		  <joint name="rear_right_flipper_joint">
+			<param name="pos_kp">10.0001</param>
+			<param name="pos_ki">1.01</param>
+			<param name="pos_kd">1.01</param>
+			<param name="pos_max_integral_error">0.1</param>
+			<command_interface name="position_pid">
+				<param name="min">-3.0</param>
+				<param name="max">3.0</param>
+				</command_interface>
+			<state_interface name="position"/>
+			<state_interface name="effort"/>
+			<state_interface name="velocity"/>
+      	</joint>
+	</ros2_control>
+	<!-- <transmission name="transmission_1">
+		<type>transmission_interface/SimpleTransmission</type>
+				<actuator name="motor_1" role="actuator1"/>
+		<joint name="left_flipper_joint"    role="joint1">
+			<hardwareInterface>PositionJointInterface</hardwareInterface>
+			<mechanical_reduction>1.0</mechanical_reduction>
+		</joint>
+	</transmission> -->
+<!--
       <joint name="right_flipper_joint">
         <command_interface name="position">
         </command_interface>
         <state_interface name="position"/>
+        <state_interface name="effort"/>
+        <state_interface name="velocity"/>
       </joint>
       <joint name="rear_left_flipper_joint">
@@ -375,15 +444,22 @@
         </command_interface>
         <state_interface name="position"/>
-      </joint>
+        <state_interface name="effort"/>
+        <state_interface name="velocity"/>
+	</joint>
       <joint name="rear_right_flipper_joint">
         <command_interface name="position">
         </command_interface>
         <state_interface name="position"/>
-      </joint>
+        <state_interface name="effort"/>
+        <state_interface name="velocity"/>
+	</joint>
     </ros2_control>
+-->
     <gazebo>
         <plugin filename="libgazebo_ros2_control.so" name="gazebo_ros2_control">
+			<!-- <robot_param>robot_description</robot_param>
+			<robot_param_node>robot_state_publisher</robot_param_node> -->
             <parameters>$(find tracked_robot_2)/config/flipper_joint.yaml</parameters>
         </plugin>
-    </gazebo> -->
+    </gazebo>
 </robot>
